File: Motorensteuerung N.17 80Ncm/Motorensteuerung.kicad_sch (KiCad schematic)
At the start: 6 parts, among them M1 17HS24-2004D-E1K, U1 TB6600, U2 AM26LV32

Commit message: Elektronik CAD Verbeesung
Parts:
- added C1: C, symbol Device:C
- added R1, R2: R, symbol Device:R
Connections:
- net at U2.1 (1B): now also M1.E4 (EA-), R1.2; no longer M1.E6 (EA-)
- net at A1.P1.21 (3V3), U2.16 (VDD), U2.4 (G): now also C1.1
- net at U2.2 (1A): now also M1.E3 (EA+), R1.1; no longer M1.E1 (EA+)
- net at U2.6 (2A): now also M1.E5 (EB+), R2.1; no longer M1.E4 (EB+)
- net at U2.7 (2B): now also M1.E6 (EB-), R2.2; no longer M1.E5 (EB-)
- net at PS2.OUT-, U2.8 (GND): now also M1.E2 (GND), C1.2; no longer M1.E3 (GND)
- net at PS2.OUT+: now also M1.E1 (VCC); no longer M1.E2 (VCC)
Other:
- note added: "Encoder"
- moved on the sheet: PS1, PS2
